File: antenna/antenna.kicad_pcb (KiCad board)
At the start: 2 copper layers, 1 part

Commit message: antennas are go
Routing:
- net Antennas: track 18.0 -> 0.00 mm
Other:
- net class Default: clearance 0.2 -> 0.2000; trace_width 0.2 -> 0.2000; via_dia 0.8 -> 0.8000; via_drill 0.4 -> 0.4000
