File: antenna/antenna_leo.kicad_pcb (KiCad board)
At the start: 2 copper layers, 1 part

Commit message: r1 RFM
Parts:
- removed ?: , X0
Other:
- net class Default: clearance 0.2000 -> 0.2; trace_width 0.2000 -> 0.2; via_dia 0.8000 -> 0.8; via_drill 0.4000 -> 0.4
