File: pcb/bikedar.kicad_pcb (KiCad board)
At the start: 4 copper layers, 50 x 50 mm, 52 parts, among them IC1 ADP3335, IC2 BGT24MTR12, IC3 AD8541, IC4 AD8226, IC5 AD8226, IC6 AD8226, IC7 AD8226, IC8 AD8541, J1 CONN_02x10, X1 M3_MOUNT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

Commit message: r1 RFM
Routing:
- net GND: track 329.7 -> 335.9 mm
- net Net-(C6-Pad2): track 20.4 -> 22.5 mm
- net Net-(C5-Pad1): track 23.3 -> 25.2 mm
- net 3v3: track 139.0 -> 140.8 mm
Other:
- net class Default: via_dia 0.6 -> 0.7
- rule via_min_size: 0.6 -> 0.7
