File: pcb/bikedar.sch (KiCad schematic (older format))
At the start: 48 parts, among them IC1 ADP3335, IC2 BGT24MTR12, IC3 AD8541, IC4 AD8226, IC5 AD8226, IC6 AD8226, IC7 AD8226, IC8 AD8541, J1 CONN_02x10, X1 M3_MOUNT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

Commit message: tidy up and add lots of gnd
Parts:
- C5, C6, R1, R2: footprint agg:0603 -> agg:0402
Changed lines of the file:
@@
 F 0 "R1" H 3650 3900 50  0000 C CNN
 F 1 "100" H 3650 3800 50  0000 C CNN
-F 2 "agg:0603" H 3600 3850 50  0001 C CNN
+F 2 "agg:0402" H 3600 3850 50  0001 C CNN
 F 3 "" H 3600 3850 50  0001 C CNN
 	1    3600 3850
@@
 F 0 "C5" H 3900 3870 50  0000 C CNN
 F 1 "1µ" H 3900 3730 50  0000 C CNN
-F 2 "agg:0603" H 3850 3800 50  0001 C CNN
+F 2 "agg:0402" H 3850 3800 50  0001 C CNN
 F 3 "" H 3850 3800 50  0001 C CNN
 	1    3850 3800
@@
 F 0 "R2" H 3650 4200 50  0000 C CNN
 F 1 "100" H 3650 4100 50  0000 C CNN
-F 2 "agg:0603" H 3600 4150 50  0001 C CNN
+F 2 "agg:0402" H 3600 4150 50  0001 C CNN
 F 3 "" H 3600 4150 50  0001 C CNN
 	1    3600 4150
@@
 F 0 "C6" H 4000 4270 50  0000 C CNN
 F 1 "1µ" H 4000 4130 50  0000 C CNN
-F 2 "agg:0603" H 3950 4200 50  0001 C CNN
+F 2 "agg:0402" H 3950 4200 50  0001 C CNN
 F 3 "" H 3950 4200 50  0001 C CNN
 	1    3950 4200

Commit message: more rf work..
Parts:
- C5, C6: value 1µ -> 100n
Other:
- note added: "RC time constants:\nWant at least 100Hz\n1/2piRC = 16kHz here, OK"
- note removed: "RC time constants TBC"
Changed lines of the file:
@@
 P 3850 3800
 F 0 "C5" H 3900 3870 50  0000 C CNN
-F 1 "1µ" H 3900 3730 50  0000 C CNN
+F 1 "100n" H 3900 3730 50  0000 C CNN
 F 2 "agg:0402" H 3850 3800 50  0001 C CNN
 F 3 "" H 3850 3800 50  0001 C CNN
@@
 P 3950 4200
 F 0 "C6" H 4000 4270 50  0000 C CNN
-F 1 "1µ" H 4000 4130 50  0000 C CNN
+F 1 "100n" H 4000 4130 50  0000 C CNN
 F 2 "agg:0402" H 3950 4200 50  0001 C CNN
 F 3 "" H 3950 4200 50  0001 C CNN
@@
 	3600 4150 3500 4150
 Text Notes 3200 3700 0    60   ~ 0
-RC time constants TBC
+RC time constants:\nWant at least 100Hz\n1/2piRC = 16kHz here, OK
 $Comp
 L R R6

Commit message: nicer balun
Parts:
- R6, R7, R8, R9: footprint agg:0603 -> agg:0402
Changed lines of the file:
@@
 F 0 "R6" H 9250 2300 50  0000 C CNN
 F 1 "5k49" H 9250 2200 50  0000 C CNN
-F 2 "agg:0603" H 9200 2250 50  0001 C CNN
+F 2 "agg:0402" H 9200 2250 50  0001 C CNN
 F 3 "" H 9200 2250 50  0001 C CNN
 	1    9200 2250
@@
 F 0 "R7" H 9250 3350 50  0000 C CNN
 F 1 "5k49" H 9250 3250 50  0000 C CNN
-F 2 "agg:0603" H 9200 3300 50  0001 C CNN
+F 2 "agg:0402" H 9200 3300 50  0001 C CNN
 F 3 "" H 9200 3300 50  0001 C CNN
 	1    9200 3300
@@
 F 0 "R8" H 9250 4400 50  0000 C CNN
 F 1 "5k49" H 9250 4300 50  0000 C CNN
-F 2 "agg:0603" H 9200 4350 50  0001 C CNN
+F 2 "agg:0402" H 9200 4350 50  0001 C CNN
 F 3 "" H 9200 4350 50  0001 C CNN
 	1    9200 4350
@@
 F 0 "R9" H 9250 5400 50  0000 C CNN
 F 1 "5k49" H 9250 5300 50  0000 C CNN
-F 2 "agg:0603" H 9200 5350 50  0001 C CNN
+F 2 "agg:0402" H 9200 5350 50  0001 C CNN
 F 3 "" H 9200 5350 50  0001 C CNN
 	1    9200 5350

Commit message: further tidying
Parts:
- added C18: 1µ, agg:0603, symbol C
Connections:
- net 3v3: now also C18.1
- net GND: now also C18.2

Commit message: further tidying
Parts:
- added C19, C20: 10µ, agg:0603, symbol C
- added D1: LED, agg:0603-LED, symbol LED
- added R14: 1k, agg:0603, symbol R
Connections:
- net 3v3: now also C19.1, C20.1, R14.1
- net GND: now also C19.2, C20.2, D1.1
- new net: D1.2, R14.2

Commit message: add mouser parts to bom (parts ordered)
Parts:
- C1, C18, C3, C7: Mouser (none) -> 81-GRM188R71C105KE5J
- C10, C11, C12, C13, C14, C16, C17, C8: Mouser (none) -> 710-885012206020
- C15, C19, C20, C4: Mouser (none) -> 81-GRM188Z71A106MA3J
- C2: Mouser (none) -> 710-885012206008
- C5, C6: Mouser (none) -> 710-885012205018
- C9: Mouser (none) -> 710-885012205025
- D1: Mouser (none) -> 710-150060VS75000
- IC1: Farnell 2067775 -> (none); Mouser (none) -> ADP3335ARMZ-3.3RL7
- IC2: Farnell 2710089 -> (none)
- IC3, IC8: Farnell 1333254 -> (none); Mouser (none) -> 584-AD8541AKSZ-R7
- IC4, IC5, IC6, IC7: Farnell 2462026 -> (none); Mouser (none) -> 584-AD8226BRMZ
- J1: Mouser (none) -> 710-61302021121
- R1, R13, R2: Mouser (none) -> 603-RC0402FR-07100RL
- R10, R11, R12, R4, R5: Mouser (none) -> 603-RC0603FR-0710KL
- R14: Mouser (none) -> 71-CRCW0603-1.0K-E3
- R3: Mouser (none) -> 660-RN731ETTP50R0F50
- R6, R7, R8, R9: Mouser (none) -> 279-CPF0402B5K49E1
Changed lines of the file:
@@
 F 2 "agg:QFN-32-BGT24MTR" H 5300 2050 50  0001 L CNN
 F 3 "http://www.infineon.com/dgdl/?fileId=db3a304339dcf4b10139df108e75025b" H 5300 1950 50  0001 L CNN
-F 4 "2710089" H 5300 1850 50  0001 L CNN "Farnell"
-F 5 "726-4MTR12E6327XUMA1" H 5300 1750 50  0001 L CNN "Mouser"
+F 4 "726-4MTR12E6327XUMA1" H 5300 1750 50  0001 L CNN "Mouser"
 	1    5700 3350
 	1    0    0    -1
@@
 F 2 "agg:MSOP-8" H 2350 850 50  0001 L CNN
 F 3 "" H 2950 850 50  0001 C CNN
-F 4 "2067775" H 2350 750 50  0001 L CNN "Farnell"
+F 4 "" H 2350 750 50  0001 L CNN "Farnell"
+F 5 "ADP3335ARMZ-3.3RL7" H 0   0   60  0001 C CNN "Mouser"
 	1    2550 1250
 	1    0    0    -1
@@
 F 2 "agg:0603" H 2950 1450 50  0001 C CNN
 F 3 "" H 2950 1450 50  0001 C CNN
+F 4 "710-885012206008" H 0   0   60  0001 C CNN "Mouser"
 	1    2950 1450
 	1    0    0    -1
@@
 F 2 "agg:0603" H 3250 1200 50  0001 C CNN
 F 3 "" H 3250 1200 50  0001 C CNN
+F 4 "81-GRM188R71C105KE5J" H 0   0   60  0001 C CNN "Mouser"
 	1    3250 1200
 	0    1    1    0
@@
 F 2 "agg:0603" H 1700 1200 50  0001 C CNN
 F 3 "" H 1700 1200 50  0001 C CNN
+F 4 "81-GRM188R71C105KE5J" H 0   0   60  0001 C CNN "Mouser"
 	1    1700 1200
 	0    1    1    0
@@
 F 2 "agg:0603" H 4700 2250 50  0001 C CNN
 F 3 "" H 4700 2250 50  0001 C CNN
+F 4 "81-GRM188R71C105KE5J" H 0   0   60  0001 C CNN "Mouser"
 	1    4700 2250
 	0    1    1    0
@@
 F 2 "agg:0603" H 4950 2250 50  0001 C CNN
 F 3 "" H 4950 2250 50  0001 C CNN
+F 4 "710-885012206020" H 0   0   60  0001 C CNN "Mouser"
 	1    4950 2250
 	0    1    1    0
@@
 F 2 "agg:0402" H 4700 4250 50  0001 C CNN
 F 3 "" H 4700 4250 50  0001 C CNN
+F 4 "660-RN731ETTP50R0F50" H 0   0   60  0001 C CNN "Mouser"
 	1    4700 4250
 	1    0    0    -1
@@
 F 2 "agg:0402" H 4950 4250 50  0001 C CNN
 F 3 "" H 4950 4250 50  0001 C CNN
+F 4 "710-885012205025" H 0   0   60  0001 C CNN "Mouser"
 	1    4950 4250
 	1    0    0    -1
@@
 F 2 "agg:MSOP-8" H 8450 1900 50  0001 L CNN
 F 3 "" H 8700 2450 50  0001 C CNN
-F 4 "2462026" H 8450 1800 50  0001 L CNN "Farnell"
+F 4 "" H 8450 1800 50  0001 L CNN "Farnell"
+F 5 "584-AD8226BRMZ" H 0   0   60  0001 C CNN "Mouser"
 	1    8650 2450
 	1    0    0    -1
@@
 F 2 "agg:0402" H 3600 3850 50  0001 C CNN
 F 3 "" H 3600 3850 50  0001 C CNN
+F 4 "603-RC0402FR-07100RL" H 0   0   60  0001 C CNN "Mouser"
 	1    3600 3850
 	1    0    0    -1
@@
 F 2 "agg:0402" H 3850 3800 50  0001 C CNN
 F 3 "" H 3850 3800 50  0001 C CNN
+F 4 "710-885012205018" H 0   0   60  0001 C CNN "Mouser"
 	1    3850 3800
 	1    0    0    -1
@@
 F 2 "agg:0402" H 3600 4150 50  0001 C CNN
 F 3 "" H 3600 4150 50  0001 C CNN
+F 4 "603-RC0402FR-07100RL" H 0   0   60  0001 C CNN "Mouser"
 	1    3600 4150
 	1    0    0    -1
@@
 F 2 "agg:0402" H 3950 4200 50  0001 C CNN
 F 3 "" H 3950 4200 50  0001 C CNN
+F 4 "710-885012205018" H 0   0   60  0001 C CNN "Mouser"
 	1    3950 4200
 	-1   0    0    1
@@
 F 2 "agg:0402" H 9200 2250 50  0001 C CNN
 F 3 "" H 9200 2250 50  0001 C CNN
+F 4 "279-CPF0402B5K49E1" H 0   0   60  0001 C CNN "Mouser"
 	1    9200 2250
 	0    -1   -1   0
@@
 F 2 "agg:0603" H 8150 2150 50  0001 C CNN
 F 3 "" H 8150 2150 50  0001 C CNN
+F 4 "710-885012206020" H 0   0   60  0001 C CNN "Mouser"
 	1    8150 2150
 	0    1    1    0
@@
 F 2 "agg:SC-70-5" H 7150 1030 50  0001 C CNN
 F 3 "" H 7050 1300 50  0001 C CNN
-F 4 "1333254" H 7150 940 50  0001 C CNN "Farnell"
+F 4 "" H 7150 940 50  0001 C CNN "Farnell"
+F 5 "584-AD8541AKSZ-R7" H 0   0   60  0001 C CNN "Mouser"
 	1    7150 1300
 	1    0    0    -1
@@
 F 2 "agg:0603" H 6600 1050 50  0001 C CNN
 F 3 "" H 6600 1050 50  0001 C CNN
+F 4 "603-RC0603FR-0710KL" H 0   0   60  0001 C CNN "Mouser"
 	1    6600 1050
 	0    1    1    0
@@
 F 2 "agg:0603" H 6600 1250 50  0001 C CNN
 F 3 "" H 6600 1250 50  0001 C CNN
+F 4 "603-RC0603FR-0710KL" H 0   0   60  0001 C CNN "Mouser"
 	1    6600 1250
 	0    1    1    0
@@
 F 2 "agg:0603" H 6900 850 50  0001 C CNN
 F 3 "" H 6900 850 50  0001 C CNN
+F 4 "710-885012206020" H 0   0   60  0001 C CNN "Mouser"
 	1    6900 850
 	0    1    1    0
@@
 F 2 "agg:0603" H 9650 2850 50  0001 C CNN
 F 3 "" H 9650 2850 50  0001 C CNN
+F 4 "81-GRM188Z71A106MA3J" H 0   0   60  0001 C CNN "Mouser"
 	1    9650 2850
 	0    1    1    0
@@
 F 2 "agg:MSOP-8" H 8450 2950 50  0001 L CNN
 F 3 "" H 8700 3500 50  0001 C CNN
-F 4 "2462026" H 8450 2850 50  0001 L CNN "Farnell"
+F 4 "" H 8450 2850 50  0001 L CNN "Farnell"
+F 5 "584-AD8226BRMZ" H 0   0   60  0001 C CNN "Mouser"
 	1    8650 3500
 	1    0    0    -1
@@
 F 2 "agg:0402" H 9200 3300 50  0001 C CNN
 F 3 "" H 9200 3300 50  0001 C CNN
+F 4 "279-CPF0402B5K49E1" H 0   0   60  0001 C CNN "Mouser"
 	1    9200 3300
 	0    -1   -1   0
@@
 F 2 "agg:0603" H 8150 3200 50  0001 C CNN
 F 3 "" H 8150 3200 50  0001 C CNN
+F 4 "710-885012206020" H 0   0   60  0001 C CNN "Mouser"
 	1    8150 3200
 	0    1    1    0
@@
 F 2 "agg:MSOP-8" H 8450 4000 50  0001 L CNN
 F 3 "" H 8700 4550 50  0001 C CNN
-F 4 "2462026" H 8450 3900 50  0001 L CNN "Farnell"
+F 4 "" H 8450 3900 50  0001 L CNN "Farnell"
+F 5 "584-AD8226BRMZ" H 0   0   60  0001 C CNN "Mouser"
 	1    8650 4550
 	1    0    0    -1
@@
 F 2 "agg:0402" H 9200 4350 50  0001 C CNN
 F 3 "" H 9200 4350 50  0001 C CNN
+F 4 "279-CPF0402B5K49E1" H 0   0   60  0001 C CNN "Mouser"
 	1    9200 4350
 	0    -1   -1   0
@@
 F 2 "agg:0603" H 8150 4250 50  0001 C CNN
 F 3 "" H 8150 4250 50  0001 C CNN
+F 4 "710-885012206020" H 0   0   60  0001 C CNN "Mouser"
 	1    8150 4250
 	0    1    1    0
@@
 F 2 "agg:MSOP-8" H 8450 5000 50  0001 L CNN
 F 3 "" H 8700 5550 50  0001 C CNN
-F 4 "2462026" H 8450 4900 50  0001 L CNN "Farnell"
+F 4 "" H 8450 4900 50  0001 L CNN "Farnell"
+F 5 "584-AD8226BRMZ" H 0   0   60  0001 C CNN "Mouser"
 	1    8650 5550
 	1    0    0    -1
@@
 F 2 "agg:0402" H 9200 5350 50  0001 C CNN
 F 3 "" H 9200 5350 50  0001 C CNN
+F 4 "279-CPF0402B5K49E1" H 0   0   60  0001 C CNN "Mouser"
 	1    9200 5350
 	0    -1   -1   0
@@
 F 2 "agg:0603" H 8150 5250 50  0001 C CNN
 F 3 "" H 8150 5250 50  0001 C CNN
+F 4 "710-885012206020" H 0   0   60  0001 C CNN "Mouser"
 	1    8150 5250
 	0    1    1    0
@@
 F 2 "agg:DIL-254P-20" H 1850 2400 50  0001 C CNN
 F 3 "" H 1850 2400 50  0001 C CNN
+F 4 "710-61302021121" H 0   0   60  0001 C CNN "Mouser"
 	1    1850 2400
 	1    0    0    -1
@@
 F 2 "agg:0603" H 2050 1400 50  0001 C CNN
 F 3 "" H 2050 1400 50  0001 C CNN
+F 4 "603-RC0603FR-0710KL" H 0   0   60  0001 C CNN "Mouser"
 	1    2050 1400
 	0    1    1    0
@@
 F 2 "agg:0603" H 9650 4900 50  0001 C CNN
 F 3 "" H 9650 4900 50  0001 C CNN
+F 4 "81-GRM188Z71A106MA3J" H 0   0   60  0001 C CNN "Mouser"
 	1    9650 4900
 	0    1    1    0
@@
 F 2 "agg:SC-70-5" H 6700 5430 50  0001 C CNN
 F 3 "" H 6600 5700 50  0001 C CNN
-F 4 "1333254" H 6700 5340 50  0001 C CNN "Farnell"
+F 4 "" H 6700 5340 50  0001 C CNN "Farnell"
+F 5 "584-AD8541AKSZ-R7" H 0   0   60  0001 C CNN "Mouser"
 	1    6700 5700
 	1    0    0    -1
@@
 F 2 "agg:0603" H 6150 5450 50  0001 C CNN
 F 3 "" H 6150 5450 50  0001 C CNN
+F 4 "603-RC0603FR-0710KL" H 0   0   60  0001 C CNN "Mouser"
 	1    6150 5450
 	0    1    1    0
@@
 F 2 "agg:0603" H 6150 5650 50  0001 C CNN
 F 3 "" H 6150 5650 50  0001 C CNN
+F 4 "603-RC0603FR-0710KL" H 0   0   60  0001 C CNN "Mouser"
 	1    6150 5650
 	0    1    1    0
@@
 F 2 "agg:0603" H 6450 5250 50  0001 C CNN
 F 3 "" H 6450 5250 50  0001 C CNN
+F 4 "710-885012206020" H 0   0   60  0001 C CNN "Mouser"
 	1    6450 5250
 	0    1    1    0
@@
 F 2 "agg:0603" H 4450 2250 50  0001 C CNN
 F 3 "" H 4450 2250 50  0001 C CNN
+F 4 "710-885012206020" H 0   0   60  0001 C CNN "Mouser"
 	1    4450 2250
 	0    1    1    0
@@
 F 2 "agg:0402" H 6450 2250 50  0001 C CNN
 F 3 "" H 6450 2250 50  0001 C CNN
+F 4 "603-RC0402FR-07100RL" H 0   0   60  0001 C CNN "Mouser"
 	1    6450 2250
 	0    1    1    0
@@
 F 2 "agg:0603" H 4200 2250 50  0001 C CNN
 F 3 "" H 4200 2250 50  0001 C CNN
+F 4 "81-GRM188R71C105KE5J" H 0   0   60  0001 C CNN "Mouser"
 	1    4200 2250
 	0    1    1    0
@@
 F 2 "agg:0603-LED" H 3850 1150 50  0001 C CNN
 F 3 "" H 3850 1150 50  0001 C CNN
+F 4 "710-150060VS75000" H 0   0   60  0001 C CNN "Mouser"
 	1    3850 1150
 	-1   0    0    1
@@
 F 2 "agg:0603" H 3500 1150 50  0001 C CNN
 F 3 "" H 3500 1150 50  0001 C CNN
+F 4 "71-CRCW0603-1.0K-E3" H 0   0   60  0001 C CNN "Mouser"
 	1    3500 1150
 	1    0    0    -1
@@
 F 2 "agg:0603" H 10000 3150 50  0001 C CNN
 F 3 "" H 10000 3150 50  0001 C CNN
+F 4 "81-GRM188Z71A106MA3J" H 0   0   60  0001 C CNN "Mouser"
 	1    10000 3150
 	0    1    1    0
@@
 F 2 "agg:0603" H 10000 5300 50  0001 C CNN
 F 3 "" H 10000 5300 50  0001 C CNN
+F 4 "81-GRM188Z71A106MA3J" H 0   0   60  0001 C CNN "Mouser"
 	1    10000 5300
 	0    1    1    0
